File: CM5_HighSpeed.kicad_sch (KiCad schematic)
At the start: 19 parts, among them J10 690-019-298-412, J12 USB3_A, J16 Conn_01x22_Female, J22 690-019-298-412, J5 Conn_01x22_Female, J6 THD-02-R, U12 RT9742SNGV, U6 AP22653W6

Commit message: first pass at layout
Connections:
- net PCIE_PWR_EN: no longer names the net of Module1.106 (PCIE_PWR_EN)
- no-connect marks 4 -> 5
Changed lines of the file:
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@@
 		(at 254 138.43)
 	)
+	(no_connect
+		(at 38.1 30.48)
+	)
 	(wire
 		(pts
@@
 	(wire
 		(pts
-			(xy 31.75 30.48) (xy 38.1 30.48)
-		)
-		(stroke
-			(width 0)
-			(type default)
-		)
-	)
-	(wire
-		(pts
 			(xy 99.06 132.08) (xy 101.6 132.08)
 		)
@@
 		)
 	)
-	(hierarchical_label "PCIE_PWR_EN"
-		(shape output)
-		(at 31.75 30.48 180)
-		(fields_autoplaced yes)
-		(effects
-			(font
-				(size 1.27 1.27)
-			)
-			(justify right)
-		)
-	)

Commit message: add LCSC part numbers, redo fan header and ps_on logic
Parts:
- C12, C13: LCSC (none) -> C92753
- C2, C7, C8: LCSC (none) -> C117956
- C3: LCSC (none) -> C189619
- J10, J22: LCSC (none) -> C720616
- J12: LCSC (none) -> C5519092
- J16, J5: LCSC (none) -> C597981
- J6: LCSC (none) -> C492419
- Module1: LCSC (none) -> C19089295
- R12: LCSC (none) -> C525579
- R6, R7, R8: LCSC (none) -> C328314
- U12: LCSC (none) -> C3235509
- U6: LCSC (none) -> C2158037
Changed lines of the file:
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@@
 			)
 		)
+		(property "LCSC" "C328314"
+			(at 207.01 110.49 0)
+			(effects
+				(font
+					(size 1.27 1.27)
+				)
+				(hide yes)
+			)
+		)
 		(pin "1"
 		)
@@
 			)
 		)
+		(property "LCSC" "C328314"
+			(at 214.63 110.49 0)
+			(effects
+				(font
+					(size 1.27 1.27)
+				)
+				(hide yes)
+			)
+		)
 		(pin "1"
 		)
@@
 			)
 		)
+		(property "LCSC" "C597981"
+			(at 156.21 50.8 0)
+			(effects
+				(font
+					(size 1.27 1.27)
+				)
+				(hide yes)
+			)
+		)
 		(pin "1"
 		)
@@
 			)
 		)
+		(property "LCSC" "C597981"
+			(at 156.21 121.92 0)
+			(effects
+				(font
+					(size 1.27 1.27)
+				)
+				(hide yes)
+			)
+		)
 		(pin "1"
 		)
@@
 			)
 		)
+		(property "LCSC" "C720616"
+			(at 264.16 50.8 0)
+			(effects
+				(font
+					(size 1.27 1.27)
+				)
+				(hide yes)
+			)
+		)
 		(pin "SH2"
 		)
@@
 			)
 		)
+		(property "LCSC" "C720616"
+			(at 264.16 123.19 0)
+			(effects
+				(font
+					(size 1.27 1.27)
+				)
+				(hide yes)
+			)
+		)
 		(pin "SH2"
 		)
@@
 			)
 		)
+		(property "LCSC" "C92753"
+			(at 229.87 151.13 0)
+			(effects
+				(font
+					(size 1.27 1.27)
+				)
+				(hide yes)
+			)
+		)
 		(pin "1"
 		)
@@
 			)
 		)
+		(property "LCSC" "C92753"
+			(at 196.85 151.13 0)
+			(effects
+				(font
+					(size 1.27 1.27)
+				)
+				(hide yes)
+			)
+		)
 		(pin "1"
 		)
@@
 			)
 		)
+		(property "LCSC" "C3235509"
+			(at 213.36 151.13 0)
+			(effects
+				(font
+					(size 1.27 1.27)
+				)
+				(hide yes)
+			)
+		)
 		(pin "1"
 		)
@@
 			)
 		)
+		(property "LCSC" "C19089295"
+			(at -71.12 86.36 0)
+			(effects
+				(font
+					(size 1.27 1.27)
+				)
+				(hide yes)
+			)
+		)
 		(pin "1"
 		)
@@
 			)
 		)
+		(property "LCSC" "C492419"
+			(at 196.85 119.38 0)
+			(effects
+				(font
+					(size 1.27 1.27)
+				)
+				(hide yes)
+			)
+		)
 		(pin "1"
 		)
@@
 			)
 		)
+		(property "LCSC" "C117956"
+			(at 100.33 181.61 0)
+			(effects
+				(font
+					(size 1.27 1.27)
+				)
+				(hide yes)
+			)
+		)
 		(pin "1"
 		)
@@
 			)
 		)
+		(property "LCSC" "C328314"
+			(at 138.43 137.16 90)
+			(effects
+				(font
+					(size 1.27 1.27)
+				)
+				(hide yes)
+			)
+		)
 		(pin "1"
 		)
@@
 			)
 		)
+		(property "LCSC" "C189619"
+			(at 87.63 181.61 0)
+			(effects
+				(font
+					(size 1.27 1.27)
+				)
+				(hide yes)
+			)
+		)
 		(pin "1"
 		)
@@
 			)
 		)
+		(property "LCSC" "C525579"
+			(at 78.74 177.8 90)
+			(effects
+				(font
+					(size 1.27 1.27)
+				)
+				(hide yes)
+			)
+		)
 		(pin "1"
 		)
@@
 			)
 		)
+		(property "LCSC" "C117956"
+			(at 110.49 181.61 0)
+			(effects
+				(font
+					(size 1.27 1.27)
+				)
+				(hide yes)
+			)
+		)
 		(pin "1"
 		)
@@
 			)
 		)
+		(property "LCSC" "C2158037"
+			(at 59.69 177.8 0)
+			(effects
+				(font
+					(size 1.27 1.27)
+				)
+				(hide yes)
+			)
+		)
 		(pin "1"
 		)
@@
 			)
 		)
+		(property "LCSC" "C5519092"
+			(at 208.28 52.07 0)
+			(effects
+				(font
+					(size 1.27 1.27)
+				)
+				(hide yes)
+			)
+		)
 		(pin "10"
 		)
@@
 			(at 29.21 180.34 0)
 			(effects
+				(font
+					(size 1.27 1.27)
+				)
+				(hide yes)
+			)
+		)
+		(property "LCSC" "C117956"
+			(at 29.21 180.34 0)
+			(effects

Commit message: update drop in replacements
Parts:
- C3: mpn (none) -> 875015119003
- J10, J22: mpn (none) -> 685119134923
- J12: mpn (none) -> 692141030100
- J6: mpn (none) -> 61300421121

Commit message: more aisler changes
Parts:
- J16, J5: mpn (none) -> 687122149022
- Module1: mpn (none) -> 10164227-1001A1RLF
Changed lines of the file:
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@@
+			)
+		)
+		(property "mpn" "687122149022"
+			(at 156.21 50.8 0)
+			(effects
+				(font
+					(size 1.27 1.27)
+				)
+				(hide yes)
 			)
 		)
@@
 			)
 		)
+		(property "mpn" "687122149022"
+			(at 156.21 121.92 0)
+			(effects
+				(font
+					(size 1.27 1.27)
+				)
+				(hide yes)
+			)
+		)
 		(pin "1"
 		)
@@
 			(at -71.12 86.36 0)
 			(effects
+				(font
+					(size 1.27 1.27)
+				)
+				(hide yes)
+			)
+		)
+		(property "mpn" "10164227-1001A1RLF"
+			(at -71.12 86.36 0)
+			(effects
